Commit message: Update vehicle geometry and track origins

File: bicycle_sim/urdf/racecar.urdf (robot description, URDF)
Before this commit: robot racecar, 8 links, 7 joints
Links:
- link ego_racecar/base_link: geometry visual box size=1.250000 1.141900 0.100000
Joints:
- joint base_to_back_left_wheel: origin xyz=0 0.120650 0.050800 -> xyz=0 0.590000 0.050800
- joint base_to_back_right_wheel: origin xyz=0 -0.120650 0.050800 -> xyz=0 -0.590000 0.050800
- joint base_to_front_left_hinge: origin xyz=0.330200 0.120650 0.050800 -> xyz=1.250000 0.590000 0.050800
- joint base_to_front_right_hinge: origin xyz=0.330200 -0.120650 0.050800 -> xyz=1.250000 -0.590000 0.050800

File: bicycle_sim/urdf/racecar.xacro (robot description, xacro)
@@ -2,10 +2,11 @@
 <!-- A model of the F1TENTH racecar for rviz -->
 <robot xmlns:xacro="http://www.ros.org/wiki/xacro" name="racecar">
-  <xacro:property name="wheelbase" value="0.3302" />
-  <xacro:property name="width" value="0.2032" />
+  <xacro:property name="wheelbase" value="1.25" />
+  <xacro:property name="track_width" value="1.18" />
   <xacro:property name="height" value="0.1" />
   <xacro:property name="ground_offset" value="0.04" />
   <xacro:property name="wheel_radius" value="0.0508" />
   <xacro:property name="wheel_length" value="0.0381" />
+  <xacro:property name="body_width" value="${track_width-wheel_length}" />
   <xacro:property name="laser_distance_from_base_link" value="0.275" />
   <xacro:property name="laser_height" value="0.05" />
@@ -25,5 +26,5 @@
       <origin xyz="${wheelbase/2} 0 ${ground_offset+height/2}"/>
       <geometry>
-        <box size="${wheelbase} ${width} ${height}"/>
+        <box size="${wheelbase} ${body_width} ${height}"/>
       </geometry>
       <material name="blue"/>
@@ -46,5 +47,5 @@
     <parent link="${car_name}/base_link"/>
     <child link="${car_name}/back_left_wheel"/>
-    <origin xyz="0 ${(wheel_length+width)/2} ${wheel_radius}"/>
+    <origin xyz="0 ${track_width/2} ${wheel_radius}"/>
     <axis xyz="0 1 0"/>
   </joint>
@@ -61,5 +62,5 @@
     <parent link="${car_name}/base_link"/>
     <child link="${car_name}/back_right_wheel"/>
-    <origin xyz="0 ${-(wheel_length+width)/2} ${wheel_radius}"/>
+    <origin xyz="0 ${-track_width/2} ${wheel_radius}"/>
     <axis xyz="0 1 0"/>
   </joint>
@@ -76,5 +77,5 @@
     <parent link="${car_name}/base_link"/>
     <child link="${car_name}/front_left_hinge"/>
-    <origin xyz="${wheelbase} ${(wheel_length+width)/2} ${wheel_radius}"/>
+    <origin xyz="${wheelbase} ${track_width/2} ${wheel_radius}"/>
     <axis xyz="0 0 1"/>
     <limit lower="-0.610865" upper="0.610865" effort="10.0" velocity="10.0"/>
@@ -98,5 +99,5 @@
     <parent link="${car_name}/base_link"/>
     <child link="${car_name}/front_right_hinge"/>
-    <origin xyz="${wheelbase} ${-(wheel_length+width)/2} ${wheel_radius}"/>
+    <origin xyz="${wheelbase} ${-track_width/2} ${wheel_radius}"/>
     <axis xyz="0 0 1"/>
     <limit lower="-0.610865" upper="0.610865" effort="10.0" velocity="10.0"/>

Commit message: Update wheel dimensions

File: bicycle_sim/urdf/racecar.urdf (robot description, URDF)
Before this commit: robot racecar, 8 links, 7 joints
Links:
- link ego_racecar/back_left_wheel: geometry visual cylinder length=0.300000 radius=0.500000
- link ego_racecar/back_right_wheel: geometry visual cylinder length=0.300000 radius=0.500000
- link ego_racecar/front_left_wheel: geometry visual cylinder length=0.300000 radius=0.500000
- link ego_racecar/front_right_wheel: geometry visual cylinder length=0.300000 radius=0.500000
Joints:
- joint base_to_back_left_wheel: origin xyz=0 0.590000 0.050800 -> xyz=0 0.590000 0.500000
- joint base_to_back_right_wheel: origin xyz=0 -0.590000 0.050800 -> xyz=0 -0.590000 0.500000
- joint base_to_front_left_hinge: origin xyz=1.250000 0.590000 0.050800 -> xyz=1.250000 0.590000 0.500000
- joint base_to_front_right_hinge: origin xyz=1.250000 -0.590000 0.050800 -> xyz=1.250000 -0.590000 0.500000

File: bicycle_sim/urdf/racecar.xacro (robot description, xacro)
@@ -6,6 +6,6 @@
   <xacro:property name="height" value="0.1" />
   <xacro:property name="ground_offset" value="0.04" />
-  <xacro:property name="wheel_radius" value="0.0508" />
-  <xacro:property name="wheel_length" value="0.0381" />
+  <xacro:property name="wheel_radius" value="0.5" />
+  <xacro:property name="wheel_length" value="0.3" />
   <xacro:property name="body_width" value="${track_width-wheel_length}" />
   <xacro:property name="laser_distance_from_base_link" value="0.275" />
